Commit message: env:dynamical test, action_param test

File: resources/models/franka_description/robots/hand.urdf (robot description, URDF)
Before this commit: robot hand, 4 links, 3 joints
Links:
- removed link tool_link
- added link panda_tcp; visual sphere radius=0.002
Joints:
- removed joint tool_joint
- added joint panda_tcp_joint: type fixed, parent panda_hand, child panda_tcp, origin xyz=0.0 0 0.1 rpy=0 0 0, axis 0 0 1

File: resources/models/franka_description/robots/hand.xacro (robot description, xacro)
@@ -47,4 +47,11 @@
       </collision>
     </link>
+    <link name="${ns}_tcp">
+      <visual>
+        <geometry>
+          <sphere radius="0.002"></sphere>
+        </geometry>
+      </visual>
+    </link>
     <joint name="${ns}_finger_joint1" type="prismatic">
       <parent link="${ns}_hand"/>
@@ -62,4 +69,10 @@
       <mimic joint="${ns}_finger_joint1" />
     </joint>
+    <joint name="${ns}_tcp_joint" type="fixed">
+        <parent link="${ns}_hand"/>
+        <child link="${ns}_tcp"/>
+        <origin rpy="0 0 0" xyz="0.0 0 0.1"/>
+        <axis xyz="0 0 1"/>
+    </joint>
   </xacro:macro>
 </robot>
